File: STM32_Blue_pill4_Kicad/STM32_Blue_pill4_Kicad.kicad_sch (KiCad schematic)
At the start: 14 parts, among them SW1 SW_SPDT, U1 STM32F103C8T6, Y1 Crystal_GND24

Commit message: Schematics is done
Parts:
- added C10, C11: 10uf, symbol Device:C
- added C12, C13: 2u2, Capacitor_SMD:C_0805_2012Metric, symbol Device:C
- added D1: LED, symbol Device:LED
- added J1: USB_B_Micro, symbol Connector:USB_B_Micro
- added J3, J4, J5: Conn_01x04_Pin, symbol Connector:Conn_01x04_Pin
- added R2, R3, R4, R5: 1K5, symbol Device:R
- added U3: AMS1117-3.3, Package_TO_SOT_SMD:SOT-223-3_TabPin2, symbol Regulator_Linear:AMS1117-3.3
Connections:
- net +3.3V: now also C13.1, D1.2 (A), J3.1 (Pin_1), J4.1 (Pin_1), J5.1 (Pin_1), R2.1, R4.1, R5.1, U3.2 (VO)
- net GND: now also Y1.2 (G), Y1.4 (G), C10.2, C11.2, C12.2, C13.2, J1.5 (GND), J3.4 (Pin_4), J4.4 (Pin_4), J5.4 (Pin_4), R3.2, U3.1 (GND)
- net HSE_IN: now also Y1.1, C10.1
- net HSE_OUT: now also Y1.3, C11.1
- net SWCLK: now also J3.3 (Pin_3)
- net SWDIO: now also J3.2 (Pin_2)
- net USB_DM+: now also J1.3 (D+), R2.2
- net USB_DM-: now also J1.2 (D-)
- net 12C_SCL: now reaches U1.21 (PB10)
- net 12C_SCL: now also J5.2 (Pin_2), R4.2
- net 12C_SDA: now reaches U1.22 (PB11)
- net 12C_SDA: now also J5.3 (Pin_3), R5.2
- net USART1_TX: now reaches U1.42 (PB6)
- net USART1_TX: now also J4.2 (Pin_2)
- net USART1_RX: now reaches U1.43 (PB7)
- net USART1_RX: now also J4.3 (Pin_3)
- new net: D1.1 (K), R3.1
- new net VBUS: C12.1, J1.1 (VBUS), U3.3 (VI)
- no-connect marks 0 -> 29
Other:
- note added: "LDO_REG"
- note added: "MICROCONTROLLER AND INTERFACES"
- note added: "The VBUS(+5V) is a power supply from USB_B_Micro and then we regulate it to +3V3 to supply the microcontroller."
- title: (none) -> STM32F103C8T6 Blue Pills
- moved on the sheet: C1, C2, C3, C4, C5, C6, C7, C8, C9, FB1, R1, SW1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

Commit message: Move to PCB design, the footprint part is done ready for layout and Routing
Parts:
- C1, C3, C4, C6, C7, C8, C9: footprint (none) -> Capacitor_SMD:C_0402_1005Metric
- C10, C11: value 10uf -> 10pf; footprint (none) -> Capacitor_SMD:C_0402_1005Metric
- C12, C13: value 2u2 -> 22uf
- C2: footprint (none) -> Capacitor_SMD:C_0201_0603Metric
- C5: footprint (none) -> Capacitor_SMD:C_0603_1608Metric
- D1: footprint (none) -> LED_SMD:LED_0603_1608Metric
- FB1: footprint (none) -> Inductor_SMD:L_0603_1608Metric
- J1: footprint (none) -> Connector_USB:USB_Micro-B_Wuerth_629105150521
- J3, J4, J5: footprint (none) -> Connector_PinHeader_2.54mm:PinHeader_1x04_P2.54mm_Vertical
- R1, R2, R3, R4, R5: footprint (none) -> Resistor_SMD:R_0402_1005Metric
- SW1: footprint (none) -> Button_Switch_THT:SW_E-Switch_EG1224_SPDT_Angled
- Y1: footprint (none) -> Crystal:Crystal_SMD_3225-4Pin_3.2x2.5mm
Changed lines of the file:
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@@
 			)
 		)
-		(property "Footprint" ""
+		(property "Footprint" "Resistor_SMD:R_0402_1005Metric"
 			(at 83.82 60.198 90)
 			(hide yes)
@@
 			)
 		)
-		(property "Footprint" ""
+		(property "Footprint" "Crystal:Crystal_SMD_3225-4Pin_3.2x2.5mm"
 			(at 59.69 82.55 0)
 			(hide yes)
@@
 			)
 		)
-		(property "Footprint" ""
+		(property "Footprint" "Capacitor_SMD:C_0402_1005Metric"
 			(at 35.2552 60.96 0)
 			(hide yes)
@@
 			)
 		)
-		(property "Footprint" ""
+		(property "Footprint" "Capacitor_SMD:C_0201_0603Metric"
 			(at 74.6252 43.18 0)
 			(hide yes)
@@
 			)
 		)
-		(property "Footprint" ""
+		(property "Footprint" "Capacitor_SMD:C_0402_1005Metric"
 			(at 143.2052 40.64 0)
 			(hide yes)
@@
 			)
 		)
-		(property "Footprint" ""
+		(property "Footprint" "Resistor_SMD:R_0402_1005Metric"
 			(at 139.192 72.39 90)
 			(hide yes)
@@
 			)
 		)
-		(property "Footprint" ""
+		(property "Footprint" "Connector_PinHeader_2.54mm:PinHeader_1x04_P2.54mm_Vertical"
 			(at 38.1 147.32 0)
 			(hide yes)
@@
 			)
 		)
-		(property "Footprint" ""
+		(property "Footprint" "Capacitor_SMD:C_0402_1005Metric"
 			(at 60.6552 43.18 0)
 			(hide yes)
@@
 			)
 		)
-		(property "Footprint" ""
+		(property "Footprint" "Capacitor_SMD:C_0603_1608Metric"
 			(at 36.5252 43.18 0)
 			(hide yes)
@@
 			)
 		)
-		(property "Value" "10uf"
+		(property "Value" "10pf"
 			(at 78.74 91.4399 0)
 			(show_name no)
@@
 			)
 		)
-		(property "Footprint" ""
+		(property "Footprint" "Capacitor_SMD:C_0402_1005Metric"
 			(at 75.8952 93.98 0)
 			(hide yes)
@@
 			)
 		)
-		(property "Footprint" ""
+		(property "Footprint" "Capacitor_SMD:C_0402_1005Metric"
 			(at 88.5952 43.18 0)
 			(hide yes)
@@
 			)
 		)
-		(property "Footprint" ""
+		(property "Footprint" "Capacitor_SMD:C_0402_1005Metric"
 			(at 168.6052 40.64 0)
 			(hide yes)
@@
 			)
 		)
-		(property "Footprint" ""
+		(property "Footprint" "Connector_PinHeader_2.54mm:PinHeader_1x04_P2.54mm_Vertical"
 			(at 172.72 102.87 0)
 			(hide yes)
@@
 			)
 		)
-		(property "Footprint" ""
+		(property "Footprint" "Button_Switch_THT:SW_E-Switch_EG1224_SPDT_Angled"
 			(at 66.04 58.42 0)
 			(hide yes)
@@
 			)
 		)
-		(property "Footprint" ""
+		(property "Footprint" "Inductor_SMD:L_0603_1608Metric"
 			(at 154.94 31.242 90)
 			(hide yes)
@@
 			)
 		)
-		(property "Value" "2u2"
+		(property "Value" "22uf"
 			(at 222.25 38.0999 0)
 			(show_name no)
@@
 			)
 		)
-		(property "Footprint" ""
+		(property "Footprint" "Resistor_SMD:R_0402_1005Metric"
 			(at 66.802 139.7 90)
 			(hide yes)
@@
 			)
 		)
-		(property "Footprint" ""
+		(property "Footprint" "Capacitor_SMD:C_0402_1005Metric"
 			(at 47.9552 43.18 0)
 			(hide yes)
@@
 			)
 		)
-		(property "Footprint" ""
+		(property "Footprint" "Connector_USB:USB_Micro-B_Wuerth_629105150521"
 			(at 165.1 80.01 0)
 			(hide yes)
@@
 			)
 		)
-		(property "Footprint" ""
+		(property "Footprint" "Capacitor_SMD:C_0402_1005Metric"
 			(at 125.4252 40.64 0)
 			(hide yes)
@@
 			)
 		)
-		(property "Footprint" ""
+		(property "Footprint" "Resistor_SMD:R_0402_1005Metric"
 			(at 267.462 36.83 90)
 			(hide yes)
@@
 			)
 		)
-		(property "Value" "10uf"
+		(property "Value" "10pf"
 			(at 48.26 91.4399 0)
 			(show_name no)
@@
 			)
 		)
-		(property "Footprint" ""
+		(property "Footprint" "Capacitor_SMD:C_0402_1005Metric"
 			(at 45.4152 93.98 0)
 			(hide yes)
@@
 			)
 		)
-		(property "Footprint" ""
+		(property "Footprint" "LED_SMD:LED_0603_1608Metric"
 			(at 261.62 33.02 0)
 			(hide yes)
@@
 			)
 		)
-		(property "Footprint" ""
+		(property "Footprint" "Connector_PinHeader_2.54mm:PinHeader_1x04_P2.54mm_Vertical"
 			(at 27.94 118.11 0)
 			(hide yes)
@@
 			)
 		)
-		(property "Value" "2u2"
+		(property "Value" "22uf"
 			(at 251.46 38.0999 0)
 			(show_name no)
@@
 			)
 		)
-		(property "Footprint" ""
+		(property "Footprint" "Resistor_SMD:R_0402_1005Metric"
 			(at 57.912 139.7 90)
 			(hide yes)

Commit message: The Layout is done , lets go for Routing
Parts:
- SW1: footprint Button_Switch_THT:SW_E-Switch_EG1224_SPDT_Angled -> Button_Switch_SMD:SW_SPDT_PCM12
Changed lines of the file:
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@@
 			)
 		)
-		(property "Footprint" "Button_Switch_THT:SW_E-Switch_EG1224_SPDT_Angled"
+		(property "Footprint" "Button_Switch_SMD:SW_SPDT_PCM12"
 			(at 66.04 58.42 0)
 			(hide yes)

Commit message: Routing of STM32 Pill is finished
Parts:
- added H1, H2, H3, H4: MountingHole, MountingHole:MountingHole_2.2mm_M2, symbol Mechanical:MountingHole
Other:
- note added: "Mounting Holes M1"
